Commit message: changes for gazebo with camera

File: src/robotic_arm_6dof/urdf/robotic_arm_6dof.urdf (robot description, URDF)
Before this commit: robot robotic_arm_6dof, 12 links, 11 joints
Links:
- added link world
- added link wrist_camera_link
- link anchor_left: mass 0.000402736212399681 -> 0.1
- link anchor_right: mass 0.00040273621239968 -> 0.1
- link base_link: mass 0.0763754463040628 -> 10.0
- link base_rotator: mass 0.0393066448790151 -> 1.0
- link elbow_Link: mass 0.0420586657729736 -> 1.0
- link end_base: mass 0.0345345547168646 -> 0.4
- link finger_left: mass 0.00220506613383814 -> 0.1
- link finger_right: mass 0.00221856156382406 -> 0.1
- link gear_left: mass 0.00146187481822585 -> 0.1
- link gear_right: mass 0.00207956891883696 -> 0.1
- link shoulder_link: mass 0.0144514859726596 -> 1.0
- link wrist_Link: mass 0.0644141323115809 -> 0.7
Joints:
- added joint world_joint: type fixed, parent world, child base_link
- added joint wrist_camera_joint: type fixed, parent wrist_Link, child wrist_camera_link, origin xyz=0.05 0 0 rpy=0 0 0
- joint anchor_left_joint: limit lower=-1.57 upper=1.57 effort=0 velocity=0 -> lower=-1.57 upper=1.57 effort=1 velocity=1
- joint anchor_right_joint: limit lower=-1.57 upper=1.57 effort=0 velocity=0 -> lower=-1.57 upper=1.57 effort=1 velocity=1
- joint elbow_joint: limit lower=-1.57 upper=1.57 effort=0 velocity=0 -> lower=-1.57 upper=1.57 effort=1 velocity=1
- joint end_joint: limit lower=-1.57 upper=1.57 effort=0 velocity=0 -> lower=-1.57 upper=1.57 effort=1 velocity=1
- joint finger_left_joint: limit lower=-1.57 upper=1.57 effort=0 velocity=0 -> lower=-1.57 upper=1.57 effort=1 velocity=1
- joint finger_right_joint: limit lower=-1.57 upper=1.57 effort=0 velocity=0 -> lower=-1.57 upper=1.57 effort=1 velocity=1
- joint gear_left_joint: limit lower=-1.57 upper=1.57 effort=0 velocity=0 -> lower=-1.57 upper=1.57 effort=1 velocity=1
- joint gear_right_joint: limit lower=-1.57 upper=1.57 effort=0 velocity=0 -> lower=-1.57 upper=1.57 effort=1 velocity=1
- joint shoulder_joint: limit lower=-1.57 upper=1.57 effort=0 velocity=0 -> lower=-1.57 upper=1.57 effort=1 velocity=1
- joint wrist_joint: limit lower=-1.57 upper=1.57 effort=0 velocity=0 -> lower=-1.57 upper=1.57 effort=1 velocity=1
